File: 3D-X2_Filament_Dryer_Modding.kicad_sch (KiCad schematic)
At the start: 70 parts, among them IC1 STM32G030F6P6, J1 24V Power In, J2 Fan, J3 Heater and Thermistor, J4 RH Sensor, J5 Conn_02x03_Odd_Even, Q1 HY1403D, Q2 CJ3400, Q3 SS8550, Q4 SS8550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

Commit message: Readme update
Connections:
- net PA3: now also R33.2; no longer R34.2
- net PB3: now also R34.2; no longer R33.2
